File: pcbs/dcconverter/dcconverter/dcconverter.kicad_pcb (KiCad board)
At the start: 2 copper layers, 41 parts, among them IC1 NCP7805TG, J1 190-9991, J2 766-6629, J3 146-8335, J4 766-6604, J5 766-6604, Q1 NGTB40N120FL2WG, Q10 398-433, Q2 FQP47P06, Q3 2SK3747-1E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

Commit message: Finish PCB for first draft of DC Converter
Parts:
- moved J4 178.6 mm to (24.1, 28.6), turned to 90 degrees
- moved J3 141.7 mm to (145.4, 148.6)
- moved Q3 140.4 mm to (79.4, 38.1)
- moved J2 137.8 mm to (163.2, 47.0), turned to 90 degrees
- moved J5 131.2 mm to (157.5, 47.0), turned to 90 degrees
- moved F2 126.9 mm to (155.6, 139.1), turned to 90 degrees
- moved R7 123.8 mm to (148.6, 40.0)
- moved R2 123.4 mm to (159.4, 52.7), turned to 270 degrees
- moved HS-Q2 123.3 mm to (110.5, 142.2)
- moved Q2 123.3 mm to (113.6, 139.6)
- moved F1 120.1 mm to (26.0, 136.5), turned to 90 degrees
- moved IC1 119.9 mm to (114.3, 37.6), turned to 0 degrees
- moved L1 119.7 mm to (66.0, 142.9), turned to 0 degrees
- moved R8 119.2 mm to (148.6, 36.8), turned to 0 degrees
- moved HS-IC1 116.4 mm to (116.8, 33.1), turned to 0 degrees
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Routing:
- net Net-(IC1-Pad3): track 15.0 -> 152.1 mm, vias 0 -> 1
- net Net-(Q5-Pad2): track 12.3 -> 137.8 mm, vias 0 -> 1
- net Net-(Q6-Pad2): track 21.9 -> 137.2 mm, vias 0 -> 1
- net Net-(Q10-Pad3): track 0.00 -> 93.7 mm, vias 0 -> 1
- net Net-(C1-Pad2): track 419.8 -> 505.8 mm, vias 1 -> 6
- net Net-(C3-Pad1): track 0.00 -> 79.2 mm, vias 0 -> 1
- net Net-(D1-Pad1): track 80.2 -> 122.4 mm
- net Net-(C4-Pad1): track 90.5 -> 49.1 mm, vias 2 -> 0
- net Net-(C1-Pad1): track 104.9 -> 145.7 mm
- net Net-(Q10-Pad2): track 0.00 -> 39.8 mm
- net Net-(D2-Pad1): track 0.00 -> 37.3 mm, vias 0 -> 2
- net Net-(F2-Pad2): track 18.7 -> 52.6 mm
- net Net-(Q3-Pad3): track 0.00 -> 33.5 mm
- net Net-(J2-Pad4): track 29.0 -> 4.71 mm
- net Net-(F1-Pad1): track 171.8 -> 149.8 mm, vias 3 -> 1
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Other:
- board outline added: 149.9 x 149.9 mm
- board text added: "+"
- board text added: "-"
- board text added: "24V"
- board text added: "5V"
- board text added: "Controller Connection Pins"
- board text added: "Fan"
- board text added: "GND"
- board text added: "Ground"
- board text added: "IGBT Control Signal (5V)"
- board text added: "IGBT ON/OFF (5V)"
- board text added: "Output Measurement 1:11"
- board text added: "Output ON/OFF (5V)"
- board text added: "Will it blend?"
