File: pcbs/rectifier/rectifier.sch (KiCad schematic (older format))
At the start: 14 parts, among them J1 494-8962, J2 494-8906, J3 422-5051, J4 422-5067

Commit message: Cleanup Symbol Library
Parts:
- C1, C2: symbol rectifier-rescue:CP-Device -> Device:CP
- D1, D2, D3, D4, D5: symbol rectifier-rescue:1N5408-Diode -> Diode:1N5408
- F1, F2: symbol rectifier-rescue:Fuse-Device -> Device:Fuse
- J1: symbol rectifier-rescue:Screw_Terminal_01x03-Connector -> Connector:Screw_Terminal_01x03
- J2: symbol rectifier-rescue:Screw_Terminal_01x02-Connector -> Connector:Screw_Terminal_01x02
- J3, J4: symbol rectifier-rescue:Conn_01x01-Connector_Generic -> Connector_Generic:Conn_01x01
- R1: symbol rectifier-rescue:R-Device -> Device:R
Changed lines of the file:
@@
 $EndDescr
 $Comp
-L rectifier-rescue:1N5408-Diode D2
+L Diode:1N5408 D2
 U 1 1 5F8757F9
 P 2400 2550
@@
 $EndComp
 $Comp
-L rectifier-rescue:1N5408-Diode D1
+L Diode:1N5408 D1
 U 1 1 5F8799EF
 P 2400 2200
@@
 $EndComp
 $Comp
-L rectifier-rescue:1N5408-Diode D4
+L Diode:1N5408 D4
 U 1 1 5F87A59A
 P 2400 3250
@@
 $EndComp
 $Comp
-L rectifier-rescue:1N5408-Diode D3
+L Diode:1N5408 D3
 U 1 1 5F87AD61
 P 2400 2900
@@
 $EndComp
 $Comp
-L rectifier-rescue:Screw_Terminal_01x03-Connector J1
+L Connector:Screw_Terminal_01x03 J1
 U 1 1 5F87C45D
 P 850 2750
@@
 	1800 2550 1800 2650
 $Comp
-L rectifier-rescue:CP-Device C1
+L Device:CP C1
 U 1 1 5F880EC9
 P 3450 2700
@@
 $EndComp
 $Comp
-L rectifier-rescue:CP-Device C2
+L Device:CP C2
 U 1 1 5F88202C
 P 4250 2700
@@
 $EndComp
 $Comp
-L rectifier-rescue:R-Device R1
+L Device:R R1
 U 1 1 5F882547
 P 3800 2200
@@
 $EndComp
 $Comp
-L rectifier-rescue:1N5408-Diode D5
+L Diode:1N5408 D5
 U 1 1 5F88410C
 P 4900 2200
@@
 $EndComp
 $Comp
-L rectifier-rescue:Fuse-Device F1
+L Device:Fuse F1
 U 1 1 5F884667
 P 1550 2650
@@
 $EndComp
 $Comp
-L rectifier-rescue:Fuse-Device F2
+L Device:Fuse F2
 U 1 1 5F886D24
 P 5450 2200
@@
 Connection ~ 3450 3250
 $Comp
-L rectifier-rescue:Screw_Terminal_01x02-Connector J2
+L Connector:Screw_Terminal_01x02 J2
 U 1 1 5F88B375
 P 6350 2700
@@
 	1050 2850 1800 2850
 $Comp
-L rectifier-rescue:Conn_01x01-Connector_Generic J4
+L Connector_Generic:Conn_01x01 J4
 U 1 1 5F88F9E1
 P 6350 3050
@@
 $EndComp
 $Comp
-L rectifier-rescue:Conn_01x01-Connector_Generic J3
+L Connector_Generic:Conn_01x01 J3
 U 1 1 5F890941
 P 6350 3250

Commit message: Minor Changes
Parts:
- C1, C2: symbol Device:CP -> rectifier-rescue:CP-Device
- D1, D2, D3, D4, D5: symbol Diode:1N5408 -> rectifier-rescue:1N5408-Diode
- F1, F2: symbol Device:Fuse -> rectifier-rescue:Fuse-Device
- J1: symbol Connector:Screw_Terminal_01x03 -> rectifier-rescue:Screw_Terminal_01x03-Connector
- J2: symbol Connector:Screw_Terminal_01x02 -> rectifier-rescue:Screw_Terminal_01x02-Connector
- J3, J4: symbol Connector_Generic:Conn_01x01 -> rectifier-rescue:Conn_01x01-Connector_Generic
- R1: symbol Device:R -> rectifier-rescue:R-Device
Changed lines of the file:
@@
 $EndDescr
 $Comp
-L Diode:1N5408 D2
+L rectifier-rescue:1N5408-Diode D2
 U 1 1 5F8757F9
 P 2400 2550
@@
 $EndComp
 $Comp
-L Diode:1N5408 D1
+L rectifier-rescue:1N5408-Diode D1
 U 1 1 5F8799EF
 P 2400 2200
@@
 $EndComp
 $Comp
-L Diode:1N5408 D4
+L rectifier-rescue:1N5408-Diode D4
 U 1 1 5F87A59A
 P 2400 3250
@@
 $EndComp
 $Comp
-L Diode:1N5408 D3
+L rectifier-rescue:1N5408-Diode D3
 U 1 1 5F87AD61
 P 2400 2900
@@
 $EndComp
 $Comp
-L Connector:Screw_Terminal_01x03 J1
+L rectifier-rescue:Screw_Terminal_01x03-Connector J1
 U 1 1 5F87C45D
 P 850 2750
@@
 	1800 2550 1800 2650
 $Comp
-L Device:CP C1
+L rectifier-rescue:CP-Device C1
 U 1 1 5F880EC9
 P 3450 2700
@@
 $EndComp
 $Comp
-L Device:CP C2
+L rectifier-rescue:CP-Device C2
 U 1 1 5F88202C
 P 4250 2700
@@
 $EndComp
 $Comp
-L Device:R R1
+L rectifier-rescue:R-Device R1
 U 1 1 5F882547
 P 3800 2200
@@
 $EndComp
 $Comp
-L Diode:1N5408 D5
+L rectifier-rescue:1N5408-Diode D5
 U 1 1 5F88410C
 P 4900 2200
@@
 $EndComp
 $Comp
-L Device:Fuse F1
+L rectifier-rescue:Fuse-Device F1
 U 1 1 5F884667
 P 1550 2650
@@
 $EndComp
 $Comp
-L Device:Fuse F2
+L rectifier-rescue:Fuse-Device F2
 U 1 1 5F886D24
 P 5450 2200
@@
 Connection ~ 3450 3250
 $Comp
-L Connector:Screw_Terminal_01x02 J2
+L rectifier-rescue:Screw_Terminal_01x02-Connector J2
 U 1 1 5F88B375
 P 6350 2700
@@
 	1050 2850 1800 2850
 $Comp
-L Connector_Generic:Conn_01x01 J4
+L rectifier-rescue:Conn_01x01-Connector_Generic J4
 U 1 1 5F88F9E1
 P 6350 3050
@@
 $EndComp
 $Comp
-L Connector_Generic:Conn_01x01 J3
+L rectifier-rescue:Conn_01x01-Connector_Generic J3
 U 1 1 5F890941
 P 6350 3250
