File: pcbs/rectifier/rectifier.sch (KiCad schematic (older format))
At the start: 14 parts, among them J1 494-8962, J2 494-8906, J3 422-5051, J4 422-5067

Commit message: Use in rectifier schematic CP symbol from custom library
Parts:
- C1, C2: symbol Device:CP -> Custom:CP-Device
Changed lines of the file:
@@
 	1800 2550 1800 2650
 $Comp
-L Device:CP C1
+L Custom:CP-Device C1
 U 1 1 5F880EC9
 P 3450 2700
@@
 $EndComp
 $Comp
-L Device:CP C2
+L Custom:CP-Device C2
 U 1 1 5F88202C
 P 4250 2700
