File: pcbs/rectifier/rectifier.sch (KiCad schematic (older format))
At the start: 14 parts, among them J1 494-8962, J2 494-8906, J3 422-5051, J4 422-5067

Commit message: Use footprint of banana socket from custom library in rectifier schematic
Parts:
- J3, J4: footprint footprints:SLB4-I90 -> Custom:SLB4-I90
Changed lines of the file:
@@
 F 0 "J4" H 6430 3092 50  0000 L CNN
 F 1 "422-5067" H 6430 3001 50  0000 L CNN
-F 2 "footprints:SLB4-I90" H 6350 3050 50  0001 C CNN
+F 2 "Custom:SLB4-I90" H 6350 3050 50  0001 C CNN
 F 3 "~" H 6350 3050 50  0001 C CNN
 	1    6350 3050
@@
 F 0 "J3" H 6430 3292 50  0000 L CNN
 F 1 "422-5051" H 6430 3201 50  0000 L CNN
-F 2 "footprints:SLB4-I90" H 6350 3250 50  0001 C CNN
+F 2 "Custom:SLB4-I90" H 6350 3250 50  0001 C CNN
 F 3 "~" H 6350 3250 50  0001 C CNN
 	1    6350 3250
