File: pcbs/dcconverter/dcconverter.kicad_pcb (KiCad board)
At the start: 4 copper layers, 160 x 100 mm, 52 parts, among them IC1 NCP7805TG, J1 190-9991, J2 Conn_01x01, J3 Conn_01x01, J4 146-8335, J5 Conn_01x01, J6 Conn_01x01, J7 483-8461, J8 483-8461, Q1 NGTB40N120FL2WG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

Commit message: Connect everything in PCB
Parts:
- moved R7 31.3 mm to (39.0, 106.5), turned to 180 degrees
- moved J7 10.5 mm to (107.0, 114.0)
- moved Q1 0.18 mm to (87.1, 30.3)
Routing:
- net Net-(Q5-Pad2): track 0.00 -> 93.7 mm
- net Net-(C3-Pad1): track 31.9 -> 108.6 mm
- net Net-(R7-Pad2): track 69.7 -> 8.65 mm
- net Net-(C1-Pad2): track 430.7 -> 434.8 mm
- net Net-(D1-Pad1): track 110.3 -> 114.2 mm
- net Net-(IC1-Pad3): track 204.5 -> 205.0 mm

Commit message: Add GND and power planes
Routing:
- added copper zone on In1.Cu, net Net-(C1-Pad2)
- added copper zone on In2.Cu, net Net-(F2-Pad1)
Changed lines of the file:
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@@
   (segment (start 15.72501 99.76101) (end 18.647601 102.683601) (width 1) (layer In2.Cu) (net 28))
   (segment (start 15.72501 65.77499) (end 15.72501 99.76101) (width 1) (layer In2.Cu) (net 28))
+  (zone (net 1) (net_name "Net-(C1-Pad2)") (layer In1.Cu) (hatch edge 0.508)
+    (connect_pads (clearance 0.508))
+    (min_thickness 0.254)
+    (fill yes (arc_segments 32) (thermal_gap 0.508) (thermal_bridge_width 0.508) (smoothing chamfer) (radius 1))
+    (polygon
+      (pts
+        (xy 173.5 17) (xy 174 103) (xy 163 103) (xy 163 114) (xy 27 114)
+        (xy 27 103) (xy 16 103) (xy 16 27) (xy 27 27) (xy 27 16)
+      )
+    )
+  )
+  (zone (net 15) (net_name "Net-(F2-Pad1)") (layer In2.Cu) (hatch edge 0.508)
+    (connect_pads (clearance 0.508))
+    (min_thickness 0.254)
+    (fill yes (arc_segments 32) (thermal_gap 0.508) (thermal_bridge_width 0.508) (smoothing chamfer) (radius 1))
+    (polygon
+      (pts
+        (xy 173.5 64) (xy 174 103) (xy 152.5 103) (xy 152.5 92) (xy 143.5 92)
+        (xy 143.5 105.5) (xy 141 108) (xy 134.5 108) (xy 134.5 95) (xy 131.5 92)
+        (xy 131.5 71) (xy 138 63.5)
+      )
+    )
+  )
 )
